File: hardware/frontend.kicad_sch (KiCad schematic)
At the start: 95 parts, among them J201 Conn_01x02, J202 Conn_01x02, J203 Conn_01x02, J204 Conn_01x02, J205 Conn_01x02, Q201 NPN, Q202 2N7002, U201 BQ769x2

Commit message: fixes
Parts:
- removed C215, C216, C217, C218, C219, C220, C221, C222, C223, C224, C225, C226, C227, C228, C229, C230, C231: 100n, Capacitor_SMD:C_0805_2012Metric, symbol Device:C_Small
- removed JP201, JP202, JP203, JP204, JP205, JP206, JP207, JP208, JP209, JP210, JP211, JP212, JP213, JP214, JP215: SolderJumper_2_Open, symbol Jumper:SolderJumper_2_Open
- removed R212, R213, R214, R215, R216, R217, R218, R219, R220, R221, R222, R223, R224, R225, R226, R227, R228: 100, Resistor_SMD:R_1206_3216Metric, symbol Device:R_Small
- U201: value BQ769x2 -> BQ7694204
Connections:
- net CELL17 is gone; now on net VC10: D202.2 (A)
- net VC11: no longer names the net of U201.5 (VC11)
- net VC12: no longer names the net of U201.4 (VC12)
- net VC13: no longer names the net of U201.3 (VC13)
- net VC14: no longer names the net of U201.2 (VC14)
- net VC15: no longer names the net of U201.1 (VC15)
- net VC16: no longer names the net of U201.48 (VC16)
- no-connect marks 14 -> 20
Other:
- moved on the sheet: C201, C202, C203, C204, C205, J201, J202, J203, J204, J205, TH201, TH202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

Commit message: add bat{en adc}
Parts:
- renumbered C206 to C201, C207 to C202, C208 to C203, C209 to C204, C210 to C205, C211 to C206, C212 to C207, C213 to C208, C214 to C209, C201 to C210, C202 to C211, C203 to C212, C204 to C213, C205 to C214, D202 to D201, D201 to D202, R229 to R207, R207 to R208, R208 to R209, R209 to R210, R210 to R211, R211 to R212

Commit message: x
Parts:
- C208: footprint Capacitor_SMD:C_0805_2012Metric -> Capacitor_SMD:C_1206_3216Metric; LCSC (none) -> C577211
- C210, C211, C212, C213, C214: footprint (none) -> Capacitor_SMD:C_0805_2012Metric
- R202, R204, R205: value 2.2k -> 2.2K
- TH201, TH202, TH203, TH205: value 10k -> 10K
Changed lines of the file:
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@@
 	)
 	(symbol
-		(lib_id "Connector_Generic:Conn_01x02")
-		(at 212.09 68.58 0)
-		(unit 1)
-		(body_style 1)
-		(exclude_from_sim no)
-		(in_bom yes)
-		(on_board yes)
-		(in_pos_files yes)
-		(dnp no)
-		(property "Reference" "J201"
-			(at 208.28 64.77 0)
-			(show_name no)
-			(do_not_autoplace no)
-			(effects
-				(font
-					(size 1.27 1.27)
-				)
-				(justify left)
-			)
-		)
-		(property "Value" "Conn_01x02"
-			(at 214.63 71.1199 0)
-			(hide yes)
-			(show_name no)
-			(do_not_autoplace no)
-			(effects
-				(font
-					(size 1.27 1.27)
-				)
-				(justify left)
-			)
-		)
-		(property "Footprint" ""
-			(at 212.09 68.58 0)
-			(hide yes)
-			(show_name no)
-			(do_not_autoplace no)
-			(effects
-				(font
-					(size 1.27 1.27)
-				)
-			)
-		)
-		(property "Datasheet" ""
-			(at 212.09 68.58 0)
-			(hide yes)
-			(show_name no)
-			(do_not_autoplace no)
-			(effects
-				(font
-					(size 1.27 1.27)
-				)
-			)
-		)
-		(property "Description" "Generic connector, single row, 01x02, script generated (kicad-library-utils/schlib/autogen/connector/)"
-			(at 212.09 68.58 0)
-			(hide yes)
-			(show_name no)
-			(do_not_autoplace no)
-			(effects
-				(font
-					(size 1.27 1.27)
-				)
-			)
-		)
-		(pin "1"
-		)
-		(pin "2"
-		)
-		(instances
-			(project "wafel-eval-board"
-				(path "/3e668e3e-3e16-4665-a807-4735962c41d3/204526d9-bdaf-4b36-9252-b50630c4791c"
-					(reference "J201")
-					(unit 1)
-				)
-			)
-		)
-	)
-	(symbol
 		(lib_id "power:GND")
 		(at 154.94 172.72 0)
@@
 			)
 		)
-		(property "Value" "10k"
+		(property "Value" "10K"
 			(at 219.71 71.4374 0)
 			(show_name no)
@@
 			)
 		)
-		(property "Footprint" "Capacitor_SMD:C_0805_2012Metric"
+		(property "Footprint" "Capacitor_SMD:C_1206_3216Metric"
 			(at 151.13 69.85 0)
 			(hide yes)
@@
 			)
 		)
+		(property "LCSC" "C577211"
+			(at 151.13 69.85 0)
+			(hide yes)
+			(show_name no)
+			(do_not_autoplace no)
+			(effects
+				(font
+					(size 1.27 1.27)
+				)
+			)
+		)
 		(pin "1"
 		)
@@
 			)
 		)
-		(property "Footprint" ""
+		(property "Footprint" "Capacitor_SMD:C_0805_2012Metric"
 			(at 195.58 71.12 0)
 			(hide yes)
@@
 			)
 		)
-		(property "Footprint" ""
+		(property "Footprint" "Capacitor_SMD:C_0805_2012Metric"
 			(at 195.58 115.57 0)
 			(hide yes)
@@
 	)
 	(symbol
+		(lib_id "Connector_Generic:Conn_01x02")
+		(at 212.09 68.58 0)
+		(unit 1)
+		(body_style 1)
+		(exclude_from_sim no)
+		(in_bom yes)
+		(on_board yes)
+		(in_pos_files yes)
+		(dnp no)
+		(property "Reference" "J201"
+			(at 208.28 64.77 0)
+			(show_name no)
+			(do_not_autoplace no)
+			(effects
+				(font
+					(size 1.27 1.27)
+				)
+				(justify left)
+			)
+		)
+		(property "Value" "Conn_01x02"
+			(at 214.63 71.1199 0)
+			(hide yes)
+			(show_name no)
+			(do_not_autoplace no)
+			(effects
+				(font
+					(size 1.27 1.27)
+				)
+				(justify left)
+			)
+		)
+		(property "Footprint" ""
+			(at 212.09 68.58 0)
+			(hide yes)
+			(show_name no)
+			(do_not_autoplace no)
+			(effects
+				(font
+					(size 1.27 1.27)
+				)
+			)
+		)
+		(property "Datasheet" ""
+			(at 212.09 68.58 0)
+			(hide yes)
+			(show_name no)
+			(do_not_autoplace no)
+			(effects
+				(font
+					(size 1.27 1.27)
+				)
+			)
+		)
+		(property "Description" "Generic connector, single row, 01x02, script generated (kicad-library-utils/schlib/autogen/connector/)"
+			(at 212.09 68.58 0)
+			(hide yes)
+			(show_name no)
+			(do_not_autoplace no)
+			(effects
+				(font
+					(size 1.27 1.27)
+				)
+			)
+		)
+		(pin "1"
+		)
+		(pin "2"
+		)
+		(instances
+			(project "wafel-eval-board"
+				(path "/3e668e3e-3e16-4665-a807-4735962c41d3/204526d9-bdaf-4b36-9252-b50630c4791c"
+					(reference "J201")
+					(unit 1)
+				)
+			)
+		)
+	)
+	(symbol
 		(lib_id "Device:R_Small")
 		(at 97.79 46.99 180)
@@
 			)
 		)
-		(property "Footprint" ""
+		(property "Footprint" "Capacitor_SMD:C_0805_2012Metric"
 			(at 229.87 68.58 0)
 			(hide yes)
@@
 			)
 		)
-		(property "Value" "2.2k"
+		(property "Value" "2.2K"
 			(at 74.93 86.36 90)
 			(show_name no)
@@
 			)
 		)
-		(property "Value" "10k"
+		(property "Value" "10K"
 			(at 219.71 117.1574 0)
 			(show_name no)
@@
 			)
 		)
-		(property "Footprint" ""
+		(property "Footprint" "Capacitor_SMD:C_0805_2012Metric"
 			(at 195.58 92.71 0)
 			(hide yes)
@@
 			)
 		)
-		(property "Value" "10k"
+		(property "Value" "10K"
 			(at 219.71 92.71 0)
 			(show_name no)
@@
 			)
 		)
-		(property "Footprint" ""
+		(property "Footprint" "Capacitor_SMD:C_0805_2012Metric"
 			(at 229.87 91.44 0)
 			(hide yes)
@@
 			)
 		)
-		(property "Value" "2.2k"
+		(property "Value" "2.2K"
 			(at 66.04 86.36 90)
 			(show_name no)
@@
 			)
 		)
-		(property "Value" "2.2k"
+		(property "Value" "2.2K"
 			(at 83.82 86.36 90)
 			(show_name no)
@@
 			)
 		)
-		(property "Value" "10k"
+		(property "Value" "10K"
 			(at 254 93.0274 0)
 			(show_name no)
