File: hardware/MCU.kicad_sch (KiCad schematic)
At the start: 16 parts, among them U801 NUCLEO-L432KC, U802 TJA1051T/3, U803 PC817

Commit message: improve can
Parts:
- removed U802: TJA1051T/3, Package_SO:SOIC-8_3.9x4.9mm_P1.27mm, symbol wafel-eval-board:CAN_Transceiver_8Pin
- removed U803: PC817, symbol Isolator:Optocoupler_DC_PhotoNPN_AKEC
- added C805: 0.1u, Capacitor_SMD:C_0805_2012Metric, symbol Device:C
- added F801: 0.1A, Fuse:Fuse_Littelfuse-NANO2-451_453, symbol Device:Fuse
- added R807: 0, Resistor_SMD:R_0805_2012Metric, symbol Device:R
- added U802: TCAN1473A, symbol wafel-eval-board:TCAN1473A
- added U804: TLP241A, Package_DIP:DIP-4_W7.62mm, symbol Relay_SolidState:TLP222A
- C804: value 0.1u -> 4.7n
- D802: value BZT52C5V6 -> ESD2CAN24-Q1; footprint Diode_SMD:D_SOD-123 -> Package_TO_SOT_SMD:SOT-23; LCSC C19077402 -> (none)
Connections:
- net +3.3V: now also F801.2, U802.5 (VIO)
- net CAN.H: now also U802.13 (CAN_H)
- net CAN.L: now also U802.12 (CAN_L)
- net GND: now also C805.2, R807.1, U802.2 (GND)
- net VESC.GND: now also U804.3
- net VESC.SW: now also U804.4
- net VESC_SW: now also U804.1
- net at U801.CN4_14 (+3V3): now also F801.1
- net ~{CAN_FAULT}: now reaches U801.CN4_6 (PA7)
- net ~{CAN_FAULT}: now also U802.8 (~{FAULT})
- net CAN_EN: now reaches U801.CN4_7 (PA6)
- net CAN_EN: now also U802.6 (EN)
- net at R806.1: now also U804.2
- net at R802.1: now also U802.14 (~{STB})
- net at C803.1, D801.1 (K), F802.1: now also C805.1, U802.10 (VSUP), U802.3 (VCC)
- net at R801.2: now also U802.1 (TXD)
- net at R803.2: now also U802.4 (RXD)
- net CAN_STB renamed CAN_N_STB
- new net: R807.2, U802.9 (WAKE)
- no-connect marks 1 -> 3
Other:
- moved on the sheet: C802, C803, D801, D802, F802, R802, R803
