File: hardware/cb_mosfet.kicad_sch (KiCad schematic)
At the start: 6 parts, among them Q1001 DMG2302U

Commit message: fixes
Parts:
- D1001: value D_Zener -> BZT52C5V6S; LCSC (none) -> C19077441
- Q1001: value DMG2302U -> DMG2302UK; LCSC (none) -> C460977
- R1001: value R_Small -> 100R 0603; LCSC (none) -> C22775
- R1002, R1003: value R_Small -> 100R 1206; LCSC (none) -> C17901
- R1004: value R_Small -> 10k 0603; LCSC (none) -> C25804
Connections:
- net vc_top is gone; now on net vc_bottom: R1001.2
- net cell_bottom: now also R1001.1
- net cell_top: no longer R1001.1
Other:
- moved on the sheet: R1004

Commit message: add bat{en adc}
Parts:
- renumbered R1002 to R1001, R1003 to R1002, R1004 to R1003, R1001 to R1004

Commit message: x
Parts:
- R1001, R1002, R1003, R1004: footprint (none) -> Resistor_SMD:R_0805_2012Metric
Changed lines of the file:
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@@
 			)
 		)
-		(property "Footprint" ""
+		(property "Footprint" "Resistor_SMD:R_0805_2012Metric"
 			(at 71.12 57.15 0)
 			(hide yes)
@@
 			)
 		)
-		(property "Footprint" ""
+		(property "Footprint" "Resistor_SMD:R_0805_2012Metric"
 			(at 99.06 69.85 0)
 			(hide yes)
@@
 			)
 		)
-		(property "Footprint" ""
+		(property "Footprint" "Resistor_SMD:R_0805_2012Metric"
 			(at 99.06 82.55 0)
 			(hide yes)
@@
 			)
 		)
-		(property "Footprint" ""
+		(property "Footprint" "Resistor_SMD:R_0805_2012Metric"
 			(at 71.12 64.77 0)
 			(hide yes)

Commit message: fix MCU pin mapping and resolve ERC conflicts
Connections:
- net cell_bottom renamed BAT_BOTTOM
- net cell_top renamed BAT_TOP
- net vc_bottom renamed VC_BOTTOM
Changed lines of the file:
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@@
 		)
 	)
-	(hierarchical_label "cell_top"
+	(hierarchical_label "BAT_TOP"
 		(shape input)
 		(at 63.5 50.8 180)
@@
 		)
 	)
-	(hierarchical_label "cell_bottom"
+	(hierarchical_label "BAT_BOTTOM"
 		(shape input)
 		(at 63.5 82.55 180)
@@
 		)
 	)
-	(hierarchical_label "vc_bottom"
+	(hierarchical_label "VC_BOTTOM"
 		(shape output)
 		(at 114.3 82.55 0)

Commit message: first layout
Parts:
- R1001, R1002: value 100R 1206 -> 100R
- R1003: value 10k 0603 -> 10k
- R1004: value 100R 0603 -> 100R
Changed lines of the file:
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@@
 			)
 		)
-		(property "Value" "100R 1206"
+		(property "Value" "100R"
 			(at 71.12 54.61 90)
 			(show_name no)
@@
 			)
 		)
-		(property "Value" "10k 0603"
+		(property "Value" "10k"
 			(at 99.06 67.31 90)
 			(show_name no)
@@
 			)
 		)
-		(property "Value" "100R 0603"
+		(property "Value" "100R"
 			(at 99.06 80.01 90)
 			(show_name no)
@@
 			)
 		)
-		(property "Value" "100R 1206"
+		(property "Value" "100R"
 			(at 71.12 62.23 90)
 			(show_name no)

Commit message: placed c mosfet
Parts:
- R1001, R1002, R1003, R1004: footprint Resistor_SMD:R_0805_2012Metric -> Resistor_SMD:R_0603_1608Metric
Changed lines of the file:
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@@
 			)
 		)
-		(property "Footprint" "Resistor_SMD:R_0805_2012Metric"
+		(property "Footprint" "Resistor_SMD:R_0603_1608Metric"
 			(at 71.12 57.15 0)
 			(hide yes)
@@
 				(path "/3e668e3e-3e16-4665-a807-4735962c41d3/fccae5ab-0edb-40a2-a80c-4f346b23f9c0/e09fd686-bb52-45eb-aef5-6296923cd8d3"
 					(reference "R1001")
-					(unit 1)
-				)
-				(path "/3e668e3e-3e16-4665-a807-4735962c41d3/fccae5ab-0edb-40a2-a80c-4f346b23f9c0/e332d889-cebe-400a-9d60-052f7f7ee759"
-					(reference "R2001")
 					(unit 1)
 				)
@@
 			)
 		)
-		(property "Footprint" "Resistor_SMD:R_0805_2012Metric"
+		(property "Footprint" "Resistor_SMD:R_0603_1608Metric"
 			(at 99.06 69.85 0)
 			(hide yes)
@@
 				(path "/3e668e3e-3e16-4665-a807-4735962c41d3/fccae5ab-0edb-40a2-a80c-4f346b23f9c0/e09fd686-bb52-45eb-aef5-6296923cd8d3"
 					(reference "R1003")
-					(unit 1)
-				)
-				(path "/3e668e3e-3e16-4665-a807-4735962c41d3/fccae5ab-0edb-40a2-a80c-4f346b23f9c0/e332d889-cebe-400a-9d60-052f7f7ee759"
-					(reference "R2003")
 					(unit 1)
 				)
@@
 				(path "/3e668e3e-3e16-4665-a807-4735962c41d3/fccae5ab-0edb-40a2-a80c-4f346b23f9c0/e09fd686-bb52-45eb-aef5-6296923cd8d3"
 					(reference "D1001")
-					(unit 1)
-				)
-				(path "/3e668e3e-3e16-4665-a807-4735962c41d3/fccae5ab-0edb-40a2-a80c-4f346b23f9c0/e332d889-cebe-400a-9d60-052f7f7ee759"
-					(reference "D2001")
 					(unit 1)
 				)
@@
 			)
 		)
-		(property "Footprint" "Resistor_SMD:R_0805_2012Metric"
+		(property "Footprint" "Resistor_SMD:R_0603_1608Metric"
 			(at 99.06 82.55 0)
 			(hide yes)
@@
 				(path "/3e668e3e-3e16-4665-a807-4735962c41d3/fccae5ab-0edb-40a2-a80c-4f346b23f9c0/e09fd686-bb52-45eb-aef5-6296923cd8d3"
 					(reference "R1004")
-					(unit 1)
-				)
-				(path "/3e668e3e-3e16-4665-a807-4735962c41d3/fccae5ab-0edb-40a2-a80c-4f346b23f9c0/e332d889-cebe-400a-9d60-052f7f7ee759"
-					(reference "R2004")
 					(unit 1)
 				)
@@
 					(unit 1)
 				)
-				(path "/3e668e3e-3e16-4665-a807-4735962c41d3/fccae5ab-0edb-40a2-a80c-4f346b23f9c0/e332d889-cebe-400a-9d60-052f7f7ee759"
-					(reference "Q2001")
-					(unit 1)
-				)
 				(path "/3e668e3e-3e16-4665-a807-4735962c41d3/fccae5ab-0edb-40a2-a80c-4f346b23f9c0/f2f1bac5-b54a-4a1b-bbb1-051fdc2ebf97"
 					(reference "Q1601")
@@
 			)
 		)
-		(property "Footprint" "Resistor_SMD:R_0805_2012Metric"
+		(property "Footprint" "Resistor_SMD:R_0603_1608Metric"
 			(at 71.12 64.77 0)
 			(hide yes)
@@
 					(unit 1)
 				)
-				(path "/3e668e3e-3e16-4665-a807-4735962c41d3/fccae5ab-0edb-40a2-a80c-4f346b23f9c0/e332d889-cebe-400a-9d60-052f7f7ee759"
-					(reference "R2002")
-					(unit 1)
-				)

Commit message: reduced BOM
Parts:
- D1001: footprint (none) -> Diode_SMD:D_SOD-323
- R1001, R1002, R1004: value 100R -> 100
