File: hardware/cb_mosfet.kicad_sch (KiCad schematic)
At the start: 6 parts, among them Q1001 DMG2302UK

Commit message: Actualize resistors size
Parts:
- R1001, R1002: footprint Resistor_SMD:R_0603_1608Metric -> Resistor_SMD:R_1206_3216Metric

Commit message: some chnages
Parts:
- Q1001: value DMG2302UK -> CJ3134K; footprint Package_TO_SOT_SMD:SOT-23 -> Package_TO_SOT_SMD:SOT-723
