File: hardware/Pre_Mosfet.kicad_sch (KiCad schematic)
At the start: 7 parts, among them Q701 PMOS

Commit message: remove jetbrains mcps, add uv in home and update flake
Parts:
- renumbered D701 to D601, D702 to D602, Q701 to Q601, R701 to R601, R702 to R602, R705 to R603, R704 to R604
Changed lines of the file:
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@@
 		(in_pos_files yes)
 		(dnp no)
-		(property "Reference" "Q701"
+		(property "Reference" "Q601"
 			(at 157.48 81.28 90)
 			(show_name no)
@@
 			(project "wafel-eval-board"
 				(path "/3e668e3e-3e16-4665-a807-4735962c41d3/5ab6bc33-292e-4a51-947f-86660ef7cdb4/1ed1b631-44e8-47fe-8167-eec9969fc398"
-					(reference "Q702")
-					(unit 1)
-				)
-				(path "/3e668e3e-3e16-4665-a807-4735962c41d3/5ab6bc33-292e-4a51-947f-86660ef7cdb4/39136857-ec23-4c0a-a04a-23d2df30ebfc"
 					(reference "Q701")
+					(unit 1)
+				)
+				(path "/3e668e3e-3e16-4665-a807-4735962c41d3/5ab6bc33-292e-4a51-947f-86660ef7cdb4/39136857-ec23-4c0a-a04a-23d2df30ebfc"
+					(reference "Q601")
 					(unit 1)
 				)
@@
 		(in_pos_files yes)
 		(dnp no)
-		(property "Reference" "R704"
+		(property "Reference" "R604"
 			(at 176.53 100.33 90)
 			(show_name no)
@@
 			(project "wafel-eval-board"
 				(path "/3e668e3e-3e16-4665-a807-4735962c41d3/5ab6bc33-292e-4a51-947f-86660ef7cdb4/1ed1b631-44e8-47fe-8167-eec9969fc398"
-					(reference "R708")
-					(unit 1)
-				)
-				(path "/3e668e3e-3e16-4665-a807-4735962c41d3/5ab6bc33-292e-4a51-947f-86660ef7cdb4/39136857-ec23-4c0a-a04a-23d2df30ebfc"
 					(reference "R704")
+					(unit 1)
+				)
+				(path "/3e668e3e-3e16-4665-a807-4735962c41d3/5ab6bc33-292e-4a51-947f-86660ef7cdb4/39136857-ec23-4c0a-a04a-23d2df30ebfc"
+					(reference "R604")
 					(unit 1)
 				)
@@
 		(in_pos_files yes)
 		(dnp no)
-		(property "Reference" "D702"
+		(property "Reference" "D602"
 			(at 151.13 99.0601 90)
 			(show_name no)
@@
 			(project "wafel-eval-board"
 				(path "/3e668e3e-3e16-4665-a807-4735962c41d3/5ab6bc33-292e-4a51-947f-86660ef7cdb4/1ed1b631-44e8-47fe-8167-eec9969fc398"
-					(reference "D704")
-					(unit 1)
-				)
-				(path "/3e668e3e-3e16-4665-a807-4735962c41d3/5ab6bc33-292e-4a51-947f-86660ef7cdb4/39136857-ec23-4c0a-a04a-23d2df30ebfc"
 					(reference "D702")
+					(unit 1)
+				)
+				(path "/3e668e3e-3e16-4665-a807-4735962c41d3/5ab6bc33-292e-4a51-947f-86660ef7cdb4/39136857-ec23-4c0a-a04a-23d2df30ebfc"
+					(reference "D602")
 					(unit 1)
 				)
@@
 		(dnp no)
 		(fields_autoplaced yes)
-		(property "Reference" "#PWR0701"
+		(property "Reference" "#PWR0601"
 			(at 124.46 135.255 0)
 			(hide yes)
@@
 			(project "wafel-eval-board"
 				(path "/3e668e3e-3e16-4665-a807-4735962c41d3/5ab6bc33-292e-4a51-947f-86660ef7cdb4/1ed1b631-44e8-47fe-8167-eec9969fc398"
-					(reference "#PWR0702")
-					(unit 1)
-				)
-				(path "/3e668e3e-3e16-4665-a807-4735962c41d3/5ab6bc33-292e-4a51-947f-86660ef7cdb4/39136857-ec23-4c0a-a04a-23d2df30ebfc"
 					(reference "#PWR0701")
+					(unit 1)
+				)
+				(path "/3e668e3e-3e16-4665-a807-4735962c41d3/5ab6bc33-292e-4a51-947f-86660ef7cdb4/39136857-ec23-4c0a-a04a-23d2df30ebfc"
+					(reference "#PWR0601")
 					(unit 1)
 				)
@@
 		(dnp no)
 		(fields_autoplaced yes)
-		(property "Reference" "R701"
+		(property "Reference" "R601"
 			(at 132.08 102.235 90)
 			(show_name no)
@@
 			(project "wafel-eval-board"
 				(path "/3e668e3e-3e16-4665-a807-4735962c41d3/5ab6bc33-292e-4a51-947f-86660ef7cdb4/1ed1b631-44e8-47fe-8167-eec9969fc398"
-					(reference "R703")
-					(unit 1)
-				)
-				(path "/3e668e3e-3e16-4665-a807-4735962c41d3/5ab6bc33-292e-4a51-947f-86660ef7cdb4/39136857-ec23-4c0a-a04a-23d2df30ebfc"
 					(reference "R701")
+					(unit 1)
+				)
+				(path "/3e668e3e-3e16-4665-a807-4735962c41d3/5ab6bc33-292e-4a51-947f-86660ef7cdb4/39136857-ec23-4c0a-a04a-23d2df30ebfc"
+					(reference "R601")
 					(unit 1)
 				)
@@
 		(dnp no)
 		(fields_autoplaced yes)
-		(property "Reference" "D701"
+		(property "Reference" "D601"
 			(at 127 118.7449 90)
 			(show_name no)
@@
 			(project "wafel-eval-board"
 				(path "/3e668e3e-3e16-4665-a807-4735962c41d3/5ab6bc33-292e-4a51-947f-86660ef7cdb4/1ed1b631-44e8-47fe-8167-eec9969fc398"
-					(reference "D703")
-					(unit 1)
-				)
-				(path "/3e668e3e-3e16-4665-a807-4735962c41d3/5ab6bc33-292e-4a51-947f-86660ef7cdb4/39136857-ec23-4c0a-a04a-23d2df30ebfc"
 					(reference "D701")
+					(unit 1)
+				)
+				(path "/3e668e3e-3e16-4665-a807-4735962c41d3/5ab6bc33-292e-4a51-947f-86660ef7cdb4/39136857-ec23-4c0a-a04a-23d2df30ebfc"
+					(reference "D601")
 					(unit 1)
 				)
@@
 		(in_pos_files yes)
 		(dnp no)
-		(property "Reference" "R705"
+		(property "Reference" "R603"
 			(at 176.53 88.9 90)
 			(show_name no)
@@
 			(project "wafel-eval-board"
 				(path "/3e668e3e-3e16-4665-a807-4735962c41d3/5ab6bc33-292e-4a51-947f-86660ef7cdb4/1ed1b631-44e8-47fe-8167-eec9969fc398"
-					(reference "R707")
-					(unit 1)
-				)
-				(path "/3e668e3e-3e16-4665-a807-4735962c41d3/5ab6bc33-292e-4a51-947f-86660ef7cdb4/39136857-ec23-4c0a-a04a-23d2df30ebfc"
-					(reference "R705")
+					(reference "R703")
+					(unit 1)
+				)
+				(path "/3e668e3e-3e16-4665-a807-4735962c41d3/5ab6bc33-292e-4a51-947f-86660ef7cdb4/39136857-ec23-4c0a-a04a-23d2df30ebfc"
+					(reference "R603")
 					(unit 1)
 				)
@@
 		(dnp no)
 		(fields_autoplaced yes)
-		(property "Reference" "R702"
+		(property "Reference" "R602"
 			(at 140.97 96.5199 0)
 			(show_name no)
@@
 			(project "wafel-eval-board"
 				(path "/3e668e3e-3e16-4665-a807-4735962c41d3/5ab6bc33-292e-4a51-947f-86660ef7cdb4/1ed1b631-44e8-47fe-8167-eec9969fc398"
-					(reference "R706")
-					(unit 1)
-				)
-				(path "/3e668e3e-3e16-4665-a807-4735962c41d3/5ab6bc33-292e-4a51-947f-86660ef7cdb4/39136857-ec23-4c0a-a04a-23d2df30ebfc"
 					(reference "R702")
 					(unit 1)
 				)
+				(path "/3e668e3e-3e16-4665-a807-4735962c41d3/5ab6bc33-292e-4a51-947f-86660ef7cdb4/39136857-ec23-4c0a-a04a-23d2df30ebfc"
+					(reference "R602")
+					(unit 1)
+				)

Commit message: x
Parts:
- R601, R602, R603, R604: footprint (none) -> Resistor_SMD:R_0805_2012Metric
Changed lines of the file:
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@@
 			)
 		)
-		(property "Footprint" ""
+		(property "Footprint" "Resistor_SMD:R_0805_2012Metric"
 			(at 176.53 92.202 90)
 			(hide yes)
@@
 			)
 		)
-		(property "Footprint" ""
+		(property "Footprint" "Resistor_SMD:R_0805_2012Metric"
 			(at 132.08 110.363 90)
 			(hide yes)
@@
 			)
 		)
-		(property "Footprint" ""
+		(property "Footprint" "Resistor_SMD:R_0805_2012Metric"
 			(at 176.53 80.772 90)
 			(hide yes)
@@
 			)
 		)
-		(property "Footprint" ""
+		(property "Footprint" "Resistor_SMD:R_0805_2012Metric"
 			(at 136.652 97.79 90)
 			(hide yes)

Commit message: placed c mosfet
Parts:
- R601, R602, R603, R604: footprint Resistor_SMD:R_0805_2012Metric -> Resistor_SMD:R_0603_1608Metric
Changed lines of the file:
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@@
 			)
 		)
-		(property "Footprint" "Resistor_SMD:R_0805_2012Metric"
+		(property "Footprint" "Resistor_SMD:R_0603_1608Metric"
 			(at 176.53 92.202 90)
 			(hide yes)
@@
 			)
 		)
-		(property "Footprint" "Resistor_SMD:R_0805_2012Metric"
+		(property "Footprint" "Resistor_SMD:R_0603_1608Metric"
 			(at 132.08 110.363 90)
 			(hide yes)
@@
 			)
 		)
-		(property "Footprint" "Resistor_SMD:R_0805_2012Metric"
+		(property "Footprint" "Resistor_SMD:R_0603_1608Metric"
 			(at 176.53 80.772 90)
 			(hide yes)
@@
 			)
 		)
-		(property "Footprint" "Resistor_SMD:R_0805_2012Metric"
+		(property "Footprint" "Resistor_SMD:R_0603_1608Metric"
 			(at 136.652 97.79 90)
 			(hide yes)

Commit message: reduced BOM
Parts:
- Q601: value PMOS -> IRFR9024

Commit message: Actualize resistors size
Parts:
- R603, R604: footprint Resistor_SMD:R_0603_1608Metric -> Resistor_SMD:R_1206_3216Metric
