File: hardware/Pre_Mosfet.kicad_sch (KiCad schematic)
At the start: 7 parts, among them Q601 IRFR9024

Commit message: Replace gate resistors with ferrite beads (600R @ 100MHz)
Parts:
- R601: value 51 -> 600R; LCSC (none) -> C139183

Commit message: Replace pre-charge/discharge MOSFETs with smaller 100V SOT-23 PJM10H01PSA
Parts:
- Q601: value IRFR9024 -> PJM10H01PSA; footprint Package_TO_SOT_SMD:TO-252-3_TabPin2 -> Package_TO_SOT_SMD:SOT-23; LCSC (none) -> C2838029

Commit message: Manually replace gate resistors with ferrite bead symbols in schematics
Parts:
- R601: symbol Device:R -> Device:L_Ferrite
