File: hardware/Mosfet_Cascade.kicad_sch (KiCad schematic)
At the start: 8 parts, among them Q401 IPB085N15NM6, Q402 IPB085N15NM6, Q403 IPB085N15NM6

Commit message: Restore robust hardware project state and clean up test files
Connections:
- net GATE: now also D401.2 (A); no longer D401.1 (K)
- net SOURCE: now also D401.1 (K); no longer D401.2 (A)
Other:
- moved on the sheet: D401

Commit message: remove jetbrains mcps, add uv in home and update flake
Parts:
- renumbered R404 to R401, R401 to R402, R402 to R403, R403 to R404
Changed lines of the file:
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@@
 		(dnp no)
 		(fields_autoplaced yes)
-		(property "Reference" "R402"
+		(property "Reference" "R403"
 			(at 135.89 91.4399 0)
 			(show_name no)
@@
 			(project "wafel-eval-board"
 				(path "/3e668e3e-3e16-4665-a807-4735962c41d3/5ab6bc33-292e-4a51-947f-86660ef7cdb4/be7298a7-6fe1-4540-a0ad-84330c0fdd5b"
-					(reference "R402")
+					(reference "R403")
 					(unit 1)
 				)
@@
 		(dnp no)
 		(fields_autoplaced yes)
-		(property "Reference" "R403"
+		(property "Reference" "R404"
 			(at 148.59 91.4399 0)
 			(show_name no)
@@
 			(project "wafel-eval-board"
 				(path "/3e668e3e-3e16-4665-a807-4735962c41d3/5ab6bc33-292e-4a51-947f-86660ef7cdb4/be7298a7-6fe1-4540-a0ad-84330c0fdd5b"
-					(reference "R403")
+					(reference "R404")
 					(unit 1)
 				)
@@
 		(dnp no)
 		(fields_autoplaced yes)
-		(property "Reference" "R401"
+		(property "Reference" "R402"
 			(at 123.19 91.4399 0)
 			(show_name no)
@@
 			(project "wafel-eval-board"
 				(path "/3e668e3e-3e16-4665-a807-4735962c41d3/5ab6bc33-292e-4a51-947f-86660ef7cdb4/be7298a7-6fe1-4540-a0ad-84330c0fdd5b"
-					(reference "R401")
+					(reference "R402")
 					(unit 1)
 				)
@@
 		(dnp no)
 		(fields_autoplaced yes)
-		(property "Reference" "R404"
+		(property "Reference" "R401"
 			(at 85.09 84.4549 0)
 			(show_name no)
@@
 			(project "wafel-eval-board"
 				(path "/3e668e3e-3e16-4665-a807-4735962c41d3/5ab6bc33-292e-4a51-947f-86660ef7cdb4/be7298a7-6fe1-4540-a0ad-84330c0fdd5b"
-					(reference "R404")
-					(unit 1)
-				)
+					(reference "R401")
+					(unit 1)
+				)

Commit message: x
Parts:
- R401, R402, R403, R404: footprint (none) -> Resistor_SMD:R_0805_2012Metric
Changed lines of the file:
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@@
 			)
 		)
-		(property "Footprint" ""
+		(property "Footprint" "Resistor_SMD:R_0805_2012Metric"
 			(at 131.572 92.71 90)
 			(hide yes)
@@
 			)
 		)
-		(property "Footprint" ""
+		(property "Footprint" "Resistor_SMD:R_0805_2012Metric"
 			(at 144.272 92.71 90)
 			(hide yes)
@@
 			)
 		)
-		(property "Footprint" ""
+		(property "Footprint" "Resistor_SMD:R_0805_2012Metric"
 			(at 118.872 92.71 90)
 			(hide yes)
@@
 			)
 		)
-		(property "Footprint" ""
+		(property "Footprint" "Resistor_SMD:R_0805_2012Metric"
 			(at 80.772 85.725 90)
 			(hide yes)

Commit message: placed c mosfet
Parts:
- R401, R402, R403, R404: footprint Resistor_SMD:R_0805_2012Metric -> Resistor_SMD:R_0603_1608Metric
Changed lines of the file:
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@@
 			)
 		)
-		(property "Footprint" "Resistor_SMD:R_0805_2012Metric"
+		(property "Footprint" "Resistor_SMD:R_0603_1608Metric"
 			(at 131.572 92.71 90)
 			(hide yes)
@@
 			)
 		)
-		(property "Footprint" "Resistor_SMD:R_0805_2012Metric"
+		(property "Footprint" "Resistor_SMD:R_0603_1608Metric"
 			(at 144.272 92.71 90)
 			(hide yes)
@@
 			)
 		)
-		(property "Footprint" "Resistor_SMD:R_0805_2012Metric"
+		(property "Footprint" "Resistor_SMD:R_0603_1608Metric"
 			(at 118.872 92.71 90)
 			(hide yes)
@@
 			)
 		)
-		(property "Footprint" "Resistor_SMD:R_0805_2012Metric"
+		(property "Footprint" "Resistor_SMD:R_0603_1608Metric"
 			(at 80.772 85.725 90)
 			(hide yes)

Commit message: Replace gate resistors with ferrite beads (600R @ 100MHz)
Parts:
- R402, R403, R404: value 51 -> 600R; LCSC (none) -> C139183

Commit message: Manually replace gate resistors with ferrite bead symbols in schematics
Parts:
- R402, R403, R404: symbol Device:R -> Device:L_Ferrite
