File: hardware/hs-mosfet.kicad_sch (KiCad schematic)
At the start: 33 parts, among them Q301 IRLML6402, Q302 2N7002K

Commit message: Update C301-C306 to 1206 100V capacitors
Parts:
- C301, C302, C303, C304, C305, C306: footprint Capacitor_SMD:C_0603_1608Metric -> Capacitor_SMD:C_1206_3216Metric; LCSC C14663 -> C110255; Voltage (none) -> 100V

Commit message: Shrink load dump Schottky diodes to SOD-323 (BAT46WS)
Parts:
- D310, D311, D312: value BAT46W -> BAT46WS; footprint Diode_SMD:D_SOD-123 -> Diode_SMD:D_SOD-323; LCSC (none) -> C7502692

Commit message: added qulon zone
Changed lines of the file:
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@@
-	)
-	(junction
-		(at 115.57 64.77)
-		(diameter 0)
-		(color 0 0 0 0)
 	)
 	(junction
@@
 	(wire
 		(pts
-			(xy 115.57 64.77) (xy 118.11 64.77)
-		)
-		(stroke
-			(width 0)
-			(type default)
-		)
-	)
-	(wire
-		(pts
 			(xy 118.11 96.52) (xy 118.11 99.06)
 		)
@@
 	(wire
 		(pts
-			(xy 115.57 52.07) (xy 115.57 64.77)
-		)
-		(stroke
-			(width 0)
-			(type default)
-		)
-	)
-	(wire
-		(pts
 			(xy 161.29 130.81) (xy 161.29 134.62)
 		)
@@
 	(wire
 		(pts
-			(xy 115.57 64.77) (xy 115.57 77.47)
+			(xy 115.57 52.07) (xy 115.57 77.47)
 		)
 		(stroke
@@
 		)
 	)
-	(label "CH"
-		(at 115.57 64.77 0)
-		(effects
-			(font
-				(size 1.27 1.27)
-			)
-			(justify left bottom)
-		)
-	)
 	(label "BAT+"
 		(at 66.04 77.47 0)
@@
 		)
 	)
-	(hierarchical_label "CH"
-		(shape output)
-		(at 118.11 64.77 0)
-		(effects
-			(font
-				(size 1.27 1.27)
-			)
-			(justify left)
-		)
-	)
